File: eagle/smartcar_shield/smartcar_shield.sch (EAGLE design)
At the start: 17 parts, among them IC1 L293D, J1 ARDUINO_R3_SHIELD

Commit message: smartcar shield rev. 1
Parts:
- added JP8, JP9: (no value), SparkFun-Connectors:M021X02_NO_SILK
- added R1, R2: 4.7KΩ, rcl:R-EU_0207/10
Connections:
- net +5V: now also JP8.1, JP8.2
- net ENABLE1: now also R1.1
- net ENABLE2: now also R2.2
- net GND: now also JP9.1, JP9.2, R1.2, R2.1
Other:
- note added: "Encoder supply"
- note added: "Free to use 5V and GND"
- note added: "L3G4200D GYROSCOPE BREAKOUT"
- note added: "Smartcar shield rev. 1"
- note added: "VBAT jumper"
Changed lines of the file:
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@@
 <?xml version="1.0" encoding="utf-8"?>
 <!DOCTYPE eagle SYSTEM "eagle.dtd">
-<eagle version="7.2.0">
+<eagle version="7.5.0">
 <drawing>
 <settings>
@@
 <setting verticaltext="up"/>
 </settings>
-<grid distance="0.1" unitdist="inch" unit="inch" style="lines" multiple="1" display="no" altdistance="0.01" altunitdist="inch" altunit="inch"/>
+<grid distance="0.05" unitdist="inch" unit="inch" style="lines" multiple="1" display="no" altdistance="0.01" altunitdist="inch" altunit="inch"/>
 <layers>
 <layer number="1" name="Top" color="4" fill="1" visible="no" active="no"/>
@@
 <layer number="95" name="Names" color="7" fill="1" visible="yes" active="yes"/>
 <layer number="96" name="Values" color="7" fill="1" visible="yes" active="yes"/>
-<layer number="97" name="Info" color="7" fill="1" visible="no" active="yes"/>
+<layer number="97" name="Info" color="7" fill="1" visible="yes" active="yes"/>
 <layer number="98" name="Guide" color="6" fill="1" visible="no" active="yes"/>
 <layer number="99" name="SpiceOrder" color="7" fill="1" visible="yes" active="yes"/>
@@
 <part name="JP4" library="SparkFun-Connectors" deviceset="M04" device="NO_SILK_ALL_ROUND"/>
 <part name="JP5" library="SparkFun-Connectors" deviceset="M04" device="NO_SILK_ALL_ROUND"/>
+<part name="R1" library="rcl" deviceset="R-EU_" device="0207/10" value="4.7KΩ"/>
+<part name="R2" library="rcl" deviceset="R-EU_" device="0207/10" value="4.7KΩ"/>
+<part name="GND14" library="supply1" deviceset="GND" device=""/>
+<part name="GND15" library="supply1" deviceset="GND" device=""/>
+<part name="P+6" library="supply1" deviceset="+5V" device=""/>
+<part name="P+7" library="supply1" deviceset="+5V" device=""/>
+<part name="GND16" library="supply1" deviceset="GND" device=""/>
+<part name="GND17" library="supply1" deviceset="GND" device=""/>
+<part name="JP8" library="SparkFun-Connectors" deviceset="M02" device="1X02_NO_SILK"/>
+<part name="JP9" library="SparkFun-Connectors" deviceset="M02" device="1X02_NO_SILK"/>
 </parts>
 <sheets>
 <sheet>
 <plain>
+<wire x1="274.32" y1="68.58" x2="294.64" y2="68.58" width="0.1524" layer="97"/>
+<wire x1="294.64" y1="68.58" x2="294.64" y2="35.56" width="0.1524" layer="97"/>
+<wire x1="294.64" y1="35.56" x2="274.32" y2="35.56" width="0.1524" layer="97"/>
+<wire x1="274.32" y1="35.56" x2="274.32" y2="68.58" width="0.1524" layer="97"/>
+<text x="293.37" y="40.64" size="1.778" layer="97" rot="R90">Encoder supply</text>
+<wire x1="114.3" y1="149.86" x2="157.48" y2="149.86" width="0.1524" layer="97"/>
+<wire x1="157.48" y1="149.86" x2="157.48" y2="115.57" width="0.1524" layer="97"/>
+<wire x1="157.48" y1="115.57" x2="114.3" y2="115.57" width="0.1524" layer="97"/>
+<wire x1="114.3" y1="115.57" x2="114.3" y2="149.86" width="0.1524" layer="97"/>
+<text x="129.54" y="144.78" size="1.778" layer="97">Free to use
+5V and GND</text>
+<wire x1="121.92" y1="104.14" x2="140.97" y2="104.14" width="0.1524" layer="97"/>
+<wire x1="140.97" y1="104.14" x2="140.97" y2="87.63" width="0.1524" layer="97"/>
+<wire x1="140.97" y1="87.63" x2="121.92" y2="87.63" width="0.1524" layer="97"/>
+<wire x1="121.92" y1="87.63" x2="121.92" y2="104.14" width="0.1524" layer="97"/>
+<text x="123.19" y="101.6" size="1.778" layer="97">VBAT jumper</text>
+<wire x1="173.99" y1="149.86" x2="284.48" y2="149.86" width="0.1524" layer="97"/>
+<wire x1="284.48" y1="149.86" x2="284.48" y2="124.46" width="0.1524" layer="97"/>
+<wire x1="284.48" y1="124.46" x2="173.99" y2="124.46" width="0.1524" layer="97"/>
+<wire x1="173.99" y1="124.46" x2="173.99" y2="149.86" width="0.1524" layer="97"/>
+<wire x1="175.26" y1="148.59" x2="283.21" y2="148.59" width="0.1524" layer="97"/>
+<wire x1="283.21" y1="148.59" x2="283.21" y2="125.73" width="0.1524" layer="97"/>
+<wire x1="283.21" y1="125.73" x2="175.26" y2="125.73" width="0.1524" layer="97"/>
+<wire x1="175.26" y1="125.73" x2="175.26" y2="148.59" width="0.1524" layer="97"/>
+<text x="229.87" y="130.81" size="5.08" layer="97" align="bottom-center">Smartcar shield
+rev. 1</text>
+<wire x1="128.27" y1="60.96" x2="184.15" y2="60.96" width="0.1524" layer="97"/>
+<wire x1="184.15" y1="60.96" x2="184.15" y2="29.21" width="0.1524" layer="97"/>
+<wire x1="184.15" y1="29.21" x2="128.27" y2="29.21" width="0.1524" layer="97"/>
+<wire x1="128.27" y1="29.21" x2="128.27" y2="60.96" width="0.1524" layer="97"/>
+<text x="156.21" y="30.48" size="2.1844" layer="97" align="bottom-center">L3G4200D GYROSCOPE BREAKOUT</text>
 </plain>
 <instances>
@@
 <instance part="JP4" gate="G$1" x="129.54" y="124.46" rot="R90"/>
 <instance part="JP5" gate="G$1" x="147.32" y="124.46" rot="R90"/>
+<instance part="R1" gate="G$1" x="223.52" y="114.3" rot="R180"/>
+<instance part="R2" gate="G$1" x="259.08" y="66.04" rot="R90"/>
+<instance part="GND14" gate="1" x="215.9" y="114.3" rot="R270"/>
+<instance part="GND15" gate="1" x="259.08" y="58.42"/>
+<instance part="P+6" gate="1" x="287.02" y="55.88" smashed="yes" rot="R180">
+<attribute name="VALUE" x="285.115" y="53.34" size="1.778" layer="96"/>
+</instance>
+<instance part="P+7" gate="1" x="287.02" y="63.5" smashed="yes">
+<attribute name="VALUE" x="288.925" y="66.04" size="1.778" layer="96" rot="R180"/>
+</instance>
+<instance part="GND16" gate="1" x="287.02" y="40.64"/>
+<instance part="GND17" gate="1" x="287.02" y="48.26" rot="R180"/>
+<instance part="JP8" gate="G$1" x="279.4" y="58.42"/>
+<instance part="JP9" gate="G$1" x="279.4" y="43.18"/>
 </instances>
 <busses>
@@
 <wire x1="132.08" y1="134.62" x2="132.08" y2="129.54" width="0.1524" layer="91"/>
 </segment>
+<segment>
+<pinref part="R1" gate="G$1" pin="2"/>
+<pinref part="GND14" gate="1" pin="GND"/>
+</segment>
+<segment>
+<pinref part="R2" gate="G$1" pin="1"/>
+<pinref part="GND15" gate="1" pin="GND"/>
+</segment>
+<segment>
+<pinref part="JP9" gate="G$1" pin="1"/>
+<pinref part="GND16" gate="1" pin="GND"/>
+</segment>
+<segment>
+<pinref part="JP9" gate="G$1" pin="2"/>
+<pinref part="GND17" gate="1" pin="GND"/>
+</segment>
 </net>
 <net name="MOTORA-OUT1" class="0">
@@
 <wire x1="149.86" y1="134.62" x2="149.86" y2="129.54" width="0.1524" layer="91"/>
 </segment>
+<segment>
+<pinref part="JP8" gate="G$1" pin="2"/>
+<pinref part="P+7" gate="1" pin="+5V"/>
+</segment>
+<segment>
+<pinref part="JP8" gate="G$1" pin="1"/>
+<pinref part="P+6" gate="1" pin="+5V"/>
+</segment>
 </net>
 <net name="12V" class="0">
@@
 <pinref part="IC1" gate="G$1" pin="1-2EN"/>
 <wire x1="193.04" y1="109.22" x2="228.6" y2="109.22" width="0.1524" layer="91"/>
+<pinref part="R1" gate="G$1" pin="1"/>
+<wire x1="228.6" y1="114.3" x2="228.6" y2="109.22" width="0.1524" layer="91"/>
 </segment>
 </net>
@@
 <pinref part="J1" gate="G$1" pin="*D9"/>
 <wire x1="190.5" y1="83.82" x2="167.64" y2="83.82" width="0.1524" layer="91"/>
+<pinref part="R2" gate="G$1" pin="2"/>
+<wire x1="259.08" y1="71.12" x2="259.08" y2="73.66" width="0.1524" layer="91"/>
 </segment>
 </net>
@@
 </schematic>
 </drawing>
+<compatibility>
+<note version="6.3" minversion="6.2.2" severity="warning">
+Since Version 6.2.2 text objects can contain more than one line,
+which will not be processed correctly with this version.
+</note>
+</compatibility>
 </eagle>
